File: HW/kicad/or_gate_interrupt.sch (KiCad schematic (older format))
At the start: 8 parts, among them P1 CONN_01X06, P2 CONN_01X03, U1 74LS32, U2 74HC02

Commit message: Added a few parts.
Parts:
- removed P2: CONN_01X03, Pin_Headers:Pin_Header_Straight_1x03, symbol CONN_01X03
- added P2, P3: CONN_01X02, Pin_Headers:Pin_Header_Straight_1x02, symbol CONN_01X02
- added U3: ESP-01v090, ESP8266:ESP-01, symbol ESP-01v090
- added U?: LT1129CST-3.3, SOT-223, symbol LT1129CST-3.3
Connections:
- net labels added: +3V3, VCC
- wire segments 48 -> 66
Changed lines of the file:
@@
 LIBS:contrib
 LIBS:valves
+LIBS:ESP8266
 EELAYER 25 0
 EELAYER END
@@
 Connection ~ 4650 5000
 Connection ~ 4500 5400
-$Comp
-L CONN_01X03 P2
-U 1 1 57E05A90
-P 8150 3900
-F 0 "P2" H 8150 4100 50  0000 C CNN
-F 1 "CONN_01X03" V 8250 3900 50  0000 C CNN
-F 2 "Pin_Headers:Pin_Header_Straight_1x03" H 8150 3900 50  0000 C CNN
-F 3 "" H 8150 3900 50  0000 C CNN
-	1    8150 3900
-	1    0    0    -1
-$EndComp
 Wire Wire Line
 	7950 3550 7950 3800
-Wire Wire Line
-	7600 3850 7950 3850
-Wire Wire Line
-	7950 3850 7950 3900
 Wire Wire Line
 	7950 4100 7950 4000
@@
 $EndComp
 Connection ~ 4200 5400
-Wire Wire Line
-	5150 4700 5150 4050
-Wire Wire Line
-	5150 4050 4800 4050
-Wire Wire Line
-	4800 4050 4800 2900
-Wire Wire Line
-	4800 2900 4450 2900
-Connection ~ 4450 2900
+$Comp
+L ESP-01v090 U3
+U 1 1 57E5BE76
+P 9200 3850
+F 0 "U3" H 9200 3750 50  0000 C CNN
+F 1 "ESP-01v090" H 9200 3950 50  0000 C CNN
+F 2 "ESP8266:ESP-01" H 9200 3850 50  0001 C CNN
+F 3 "" H 9200 3850 50  0001 C CNN
+	1    9200 3850
+	-1   0    0    1
+$EndComp
+Wire Wire Line
+	7950 3800 8250 3800
+Wire Wire Line
+	8250 3900 8050 3900
+Wire Wire Line
+	8050 3900 8050 4000
+Wire Wire Line
+	8050 4000 7950 4000
+Wire Wire Line
+	7600 3850 7800 3850
+Wire Wire Line
+	7800 3850 7800 3350
+Wire Wire Line
+	7800 3350 10300 3350
+Wire Wire Line
+	10300 3350 10300 3800
+Wire Wire Line
+	10300 3800 10150 3800
+$Comp
+L GND #PWR05
+U 1 1 57E5C006
+P 8250 4400
+F 0 "#PWR05" H 8250 4150 50  0001 C CNN
+F 1 "GND" H 8250 4250 50  0000 C CNN
+F 2 "" H 8250 4400 50  0000 C CNN
+F 3 "" H 8250 4400 50  0000 C CNN
+	1    8250 4400
+	1    0    0    -1
+$EndComp
+$Comp
+L +3V3 #PWR06
+U 1 1 57E5C107
+P 10150 3600
+F 0 "#PWR06" H 10150 3450 50  0001 C CNN
+F 1 "+3V3" H 10150 3740 50  0000 C CNN
+F 2 "" H 10150 3600 50  0000 C CNN
+F 3 "" H 10150 3600 50  0000 C CNN
+	1    10150 3600
+	1    0    0    -1
+$EndComp
+Wire Wire Line
+	10150 3600 10150 3700
+Wire Wire Line
+	8250 4000 8250 4400
+$Comp
+L CONN_01X02 P2
+U 1 1 57E5C3BD
+P 8050 4600
+F 0 "P2" H 8050 4750 50  0000 C CNN
+F 1 "CONN_01X02" V 8150 4600 50  0000 C CNN
+F 2 "Pin_Headers:Pin_Header_Straight_1x02" H 8050 4600 50  0000 C CNN
+F 3 "" H 8050 4600 50  0000 C CNN
+	1    8050 4600
+	0    1    1    0
+$EndComp
+Wire Wire Line
+	8100 4400 8100 4200
+Wire Wire Line
+	8100 4200 8250 4200
+Connection ~ 8250 4200
+Wire Wire Line
+	8000 4400 8000 3800
+Connection ~ 8000 3800
+$Comp
+L CONN_01X02 P3
+U 1 1 57E5C4F4
+P 9100 2800
+F 0 "P3" H 9100 2950 50  0000 C CNN
+F 1 "CONN_01X02" V 9200 2800 50  0000 C CNN
+F 2 "Pin_Headers:Pin_Header_Straight_1x02" H 9100 2800 50  0000 C CNN
+F 3 "" H 9100 2800 50  0000 C CNN
+	1    9100 2800
+	0    -1   -1   0
+$EndComp
+Wire Wire Line
+	8250 3700 8250 3100
+Wire Wire Line
+	8250 3100 9050 3100
+Wire Wire Line
+	9050 3100 9050 3000
+Wire Wire Line
+	9150 3000 9150 3100
+Wire Wire Line
+	9150 3100 10450 3100
+Wire Wire Line
+	10450 3100 10450 4000
+Wire Wire Line
+	10450 4000 10150 4000
+Wire Wire Line
+	10150 3900 10200 3900
+Wire Wire Line
+	10200 3900 10200 3650
+Wire Wire Line
+	10200 3650 10150 3650
+Connection ~ 10150 3650
+Text Label 4450 3100 1    60   ~ 0
+VCC
+Text Label 10200 3950 0    60   ~ 0
+VCC
+Text Label 8250 4150 1    60   ~ 0
+GND
+Text Label 4200 5050 1    60   ~ 0
+GND
+$Comp
+L LT1129CST-3.3 U?
+U 1 1 57E5E51E
+P 3100 2750
+F 0 "U?" H 2850 2950 50  0000 C CNN
+F 1 "LT1129CST-3.3" H 3250 2950 50  0000 C CNN
+F 2 "SOT-223" H 3100 2850 50  0000 C CIN
+F 3 "" H 3100 2750 50  0000 C CNN
+	1    3100 2750
+	1    0    0    -1
+$EndComp
 $EndSCHEMATC

Commit message: Updated a few layout things.
Parts:
- added C1: CP, Capacitors_ThroughHole:C_Radial_D6.3_L11.2_P2.5, symbol CP
- gave numbers to parts that had none: 1
Connections:
- net +3V3: now also U4.3 (OUT), C1.1; no longer P1.6 (P6)
- net GND: now also U4.2 (GND), C1.2
- net at U4.1 (VIN): now also P1.6 (P6)
Other:
- moved on the sheet: U4
Changed lines of the file:
@@
 L +3.3V #VCC01
 U 1 1 57E064D6
-P 4450 2700
-F 0 "#VCC01" H 4450 2550 50  0001 C CNN
-F 1 "+3.3V" H 4450 2840 50  0000 C CNN
-F 2 "" H 4450 2700 50  0000 C CNN
-F 3 "" H 4450 2700 50  0000 C CNN
-	1    4450 2700
-	1    0    0    -1
-$EndComp
-Wire Wire Line
-	4450 2700 4450 3100
-Wire Wire Line
-	4450 3100 4200 3100
+P 5800 2200
+F 0 "#VCC01" H 5800 2050 50  0001 C CNN
+F 1 "+3.3V" H 5800 2340 50  0000 C CNN
+F 2 "" H 5800 2200 50  0000 C CNN
+F 3 "" H 5800 2200 50  0000 C CNN
+	1    5800 2200
+	1    0    0    -1
+$EndComp
 $Comp
 L GND #GND02
@@
 L PWR_FLAG #VCC03
 U 1 1 57E06E87
-P 4300 3000
-F 0 "#VCC03" H 4300 3095 50  0001 C CNN
-F 1 "PWR_FLAG" H 4300 3180 50  0000 C CNN
-F 2 "" H 4300 3000 50  0000 C CNN
-F 3 "" H 4300 3000 50  0000 C CNN
-	1    4300 3000
-	1    0    0    -1
-$EndComp
-Wire Wire Line
-	4300 3000 4300 3100
-Connection ~ 4300 3100
+P 4250 2200
+F 0 "#VCC03" H 4250 2295 50  0001 C CNN
+F 1 "PWR_FLAG" H 4250 2380 50  0000 C CNN
+F 2 "" H 4250 2200 50  0000 C CNN
+F 3 "" H 4250 2200 50  0000 C CNN
+	1    4250 2200
+	1    0    0    -1
+$EndComp
 $Comp
 L PWR_FLAG #GND04
@@
 	10200 3650 10150 3650
 Connection ~ 10150 3650
-Text Label 4450 3100 1    60   ~ 0
-VCC
 Text Label 10200 3950 0    60   ~ 0
 VCC
@@
 GND
 $Comp
-L LT1129CST-3.3 U?
+L LT1129CST-3.3 U4
 U 1 1 57E5E51E
-P 3100 2750
-F 0 "U?" H 2850 2950 50  0000 C CNN
-F 1 "LT1129CST-3.3" H 3250 2950 50  0000 C CNN
-F 2 "SOT-223" H 3100 2850 50  0000 C CIN
-F 3 "" H 3100 2750 50  0000 C CNN
-	1    3100 2750
-	1    0    0    -1
-$EndComp
+P 4800 2300
+F 0 "U4" H 4550 2500 50  0000 C CNN
+F 1 "LT1129CST-3.3" H 4950 2500 50  0000 C CNN
+F 2 "SOT-223" H 4800 2400 50  0000 C CIN
+F 3 "" H 4800 2300 50  0000 C CNN
+	1    4800 2300
+	1    0    0    -1
+$EndComp
+Wire Wire Line
+	5250 2250 5800 2250
+Wire Wire Line
+	5800 2250 5800 2200
+Wire Wire Line
+	4350 2250 4250 2250
+Wire Wire Line
+	4250 2200 4250 3100
+Wire Wire Line
+	4250 3100 4200 3100
+Wire Wire Line
+	4200 3800 4400 3800
+Wire Wire Line
+	4400 3800 4400 2700
+Wire Wire Line
+	4400 2700 5000 2700
+Wire Wire Line
+	4800 2700 4800 2600
+Connection ~ 4200 3800
+$Comp
+L CP C1
+U 1 1 57E9B7FD
+P 5150 2700
+F 0 "C1" H 5175 2800 50  0000 L CNN
+F 1 "CP" H 5175 2600 50  0000 L CNN
+F 2 "Capacitors_ThroughHole:C_Radial_D6.3_L11.2_P2.5" H 5188 2550 50  0000 C CNN
+F 3 "" H 5150 2700 50  0000 C CNN
+	1    5150 2700
+	0    1    1    0
+$EndComp
+Connection ~ 4800 2700
+Wire Wire Line
+	5300 2700 5300 2250
+Connection ~ 5300 2250
+Connection ~ 4250 2250
+Text Label 5400 2250 0    60   ~ 0
+VCC
 $EndSCHEMATC

Commit message: Updating layout.
Parts:
- C1: value CP -> 100uF; footprint Capacitors_ThroughHole:C_Radial_D6.3_L11.2_P2.5 -> Capacitors_SMD:C_1210_HandSoldering; MN (none) -> TAJB107M006RNJ
- R1, R2, R3, R4: value R -> 1K
Changed lines of the file:
@@
 P 5600 3000
 F 0 "R1" V 5680 3000 50  0000 C CNN
-F 1 "R" V 5600 3000 50  0000 C CNN
+F 1 "1K" V 5600 3000 50  0000 C CNN
 F 2 "Resistors_SMD:R_1206_HandSoldering" V 5530 3000 50  0000 C CNN
 F 3 "" H 5600 3000 50  0000 C CNN
@@
 P 4650 3600
 F 0 "R3" V 4730 3600 50  0000 C CNN
-F 1 "R" V 4650 3600 50  0000 C CNN
+F 1 "1K" V 4650 3600 50  0000 C CNN
 F 2 "Resistors_SMD:R_1206_HandSoldering" V 4580 3600 50  0000 C CNN
 F 3 "" H 4650 3600 50  0000 C CNN
@@
 P 5700 4550
 F 0 "R2" V 5780 4550 50  0000 C CNN
-F 1 "R" V 5700 4550 50  0000 C CNN
+F 1 "1K" V 5700 4550 50  0000 C CNN
 F 2 "Resistors_SMD:R_1206_HandSoldering" V 5630 4550 50  0000 C CNN
 F 3 "" H 5700 4550 50  0000 C CNN
@@
 P 4500 5250
 F 0 "R4" V 4580 5250 50  0000 C CNN
-F 1 "R" V 4500 5250 50  0000 C CNN
+F 1 "1K" V 4500 5250 50  0000 C CNN
 F 2 "Resistors_SMD:R_1206_HandSoldering" V 4430 5250 50  0000 C CNN
 F 3 "" H 4500 5250 50  0000 C CNN
@@
 P 5150 2700
 F 0 "C1" H 5175 2800 50  0000 L CNN
-F 1 "CP" H 5175 2600 50  0000 L CNN
-F 2 "Capacitors_ThroughHole:C_Radial_D6.3_L11.2_P2.5" H 5188 2550 50  0000 C CNN
-F 3 "" H 5150 2700 50  0000 C CNN
+F 1 "100uF" H 5175 2600 50  0000 L CNN
+F 2 "Capacitors_SMD:C_1210_HandSoldering" H 5188 2550 50  0000 C CNN
+F 3 "http://datasheets.avx.com/TAJ.pdf" H 5150 2700 50  0000 C CNN
+F 4 "TAJB107M006RNJ" H 5150 2700 60  0001 C CNN "MN"
 	1    5150 2700
 	0    1    1    0

Commit message: Updated BOM.  Changed cap to smt.
Parts:
- C1: footprint Capacitors_SMD:C_1210_HandSoldering -> Capacitors_SMD:C_1206_HandSoldering
Changed lines of the file:
@@
 LIBS:valves
 LIBS:ESP8266
+LIBS:or_gate_interrupt-cache
 EELAYER 25 0
 EELAYER END
@@
 F 0 "C1" H 5175 2800 50  0000 L CNN
 F 1 "100uF" H 5175 2600 50  0000 L CNN
-F 2 "Capacitors_SMD:C_1210_HandSoldering" H 5188 2550 50  0000 C CNN
+F 2 "Capacitors_SMD:C_1206_HandSoldering" H 5188 2550 50  0000 C CNN
 F 3 "http://datasheets.avx.com/TAJ.pdf" H 5150 2700 50  0000 C CNN
 F 4 "TAJB107M006RNJ" H 5150 2700 60  0001 C CNN "MN"

Commit message: Rerouted with new resistor size.  Need to shrink board.
Parts:
- P1: value CONN_01X06 -> G_G_G_I1_I2_V
- P3: value CONN_01X02 -> Rx_Tx
- R1, R2, R3, R4: footprint Resistors_SMD:R_1206_HandSoldering -> Resistors_SMD:R_0805_HandSoldering
Changed lines of the file:
@@
 P 4000 3350
 F 0 "P1" H 4000 3700 50  0000 C CNN
-F 1 "CONN_01X06" V 4100 3350 50  0000 C CNN
+F 1 "G_G_G_I1_I2_V" V 4100 3350 50  0000 C CNN
 F 2 "Pin_Headers:Pin_Header_Straight_1x06" H 4000 3350 50  0000 C CNN
 F 3 "" H 4000 3350 50  0000 C CNN
@@
 F 0 "R1" V 5680 3000 50  0000 C CNN
 F 1 "1K" V 5600 3000 50  0000 C CNN
-F 2 "Resistors_SMD:R_1206_HandSoldering" V 5530 3000 50  0000 C CNN
+F 2 "Resistors_SMD:R_0805_HandSoldering" V 5530 3000 50  0000 C CNN
 F 3 "" H 5600 3000 50  0000 C CNN
 	1    5600 3000
@@
 F 0 "R3" V 4730 3600 50  0000 C CNN
 F 1 "1K" V 4650 3600 50  0000 C CNN
-F 2 "Resistors_SMD:R_1206_HandSoldering" V 4580 3600 50  0000 C CNN
+F 2 "Resistors_SMD:R_0805_HandSoldering" V 4580 3600 50  0000 C CNN
 F 3 "" H 4650 3600 50  0000 C CNN
 	1    4650 3600
@@
 F 0 "R2" V 5780 4550 50  0000 C CNN
 F 1 "1K" V 5700 4550 50  0000 C CNN
-F 2 "Resistors_SMD:R_1206_HandSoldering" V 5630 4550 50  0000 C CNN
+F 2 "Resistors_SMD:R_0805_HandSoldering" V 5630 4550 50  0000 C CNN
 F 3 "" H 5700 4550 50  0000 C CNN
 	1    5700 4550
@@
 F 0 "R4" V 4580 5250 50  0000 C CNN
 F 1 "1K" V 4500 5250 50  0000 C CNN
-F 2 "Resistors_SMD:R_1206_HandSoldering" V 4430 5250 50  0000 C CNN
+F 2 "Resistors_SMD:R_0805_HandSoldering" V 4430 5250 50  0000 C CNN
 F 3 "" H 4500 5250 50  0000 C CNN
 	1    4500 5250
@@
 P 9100 2800
 F 0 "P3" H 9100 2950 50  0000 C CNN
-F 1 "CONN_01X02" V 9200 2800 50  0000 C CNN
+F 1 "Rx_Tx" V 9200 2800 50  0000 C CNN
 F 2 "Pin_Headers:Pin_Header_Straight_1x02" H 9100 2800 50  0000 C CNN
 F 3 "" H 9100 2800 50  0000 C CNN

Commit message: Updating some changes.
Parts:
- P2: value CONN_01X02 -> GND_GP0
- U4: SN (none) -> MCP1825S-3302E/DB
Changed lines of the file:
@@
 P 8050 4600
 F 0 "P2" H 8050 4750 50  0000 C CNN
-F 1 "CONN_01X02" V 8150 4600 50  0000 C CNN
+F 1 "GND_GP0" V 8150 4600 50  0000 C CNN
 F 2 "Pin_Headers:Pin_Header_Straight_1x02" H 8050 4600 50  0000 C CNN
 F 3 "" H 8050 4600 50  0000 C CNN
@@
 F 2 "SOT-223" H 4800 2400 50  0000 C CIN
 F 3 "" H 4800 2300 50  0000 C CNN
+F 4 "MCP1825S-3302E/DB" H 4800 2300 60  0001 C CNN "SN"
 	1    4800 2300
 	1    0    0    -1
