File: HW/kicad/or_gate_interrupt.kicad_pcb (KiCad board)
At the start: 2 copper layers, 27.9 x 47 mm, 12 parts, among them P1 V_I1_I2_G_G_G, P2 CONN_01X02, P3 Rx_Tx, U1 74LS32, U2 74HC02, U3 ESP-01v090, U4 LT1129CST-3.3

Commit message: Updating some changes.
Parts:
- P1: value V_I1_I2_G_G_G -> G_G_G_I1_I2_V
- P2: value CONN_01X02 -> GND_GP0
Other:
- board size 27.9 x 47 mm -> 24.4 x 45.2 mm
Changed lines of the file:
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@@
     (links 32)
     (no_connects 0)
-    (area 110.489499 64.968 151.51 118.205)
+    (area 112.521499 71.881499 136.906501 117.094501)
     (thickness 1.6)
-    (drawings 6)
+    (drawings 8)
     (tracks 152)
     (zones 0)
@@
       (effects (font (size 1 1) (thickness 0.15)))
     )
-    (fp_text value V_I1_I2_G_G_G (at -1.651 7.747 90) (layer F.Fab)
+    (fp_text value G_G_G_I1_I2_V (at -1.651 7.747 90) (layer F.Fab)
       (effects (font (size 1 1) (thickness 0.15)))
     )
@@
       (effects (font (size 1 1) (thickness 0.15)))
     )
-    (fp_text value 74HC02 (at 0 4.2) (layer F.Fab)
+    (fp_text value 74HC02 (at 1.524 0 90) (layer F.Fab)
       (effects (font (size 1 1) (thickness 0.15)))
     )
@@
       (effects (font (size 1 1) (thickness 0.15)))
     )
-    (fp_text value Rx_Tx (at -3.81 -1.27) (layer F.Fab)
+    (fp_text value Rx_Tx (at -2.032 1.524 90) (layer F.Fab)
       (effects (font (size 1 1) (thickness 0.15)))
     )
@@
       (effects (font (size 1 1) (thickness 0.15)))
     )
-    (fp_text value CONN_01X02 (at -2.54 -2.54 180) (layer F.Fab)
+    (fp_text value GND_GP0 (at 2.032 0.762 270) (layer F.Fab)
       (effects (font (size 1 1) (thickness 0.15)))
     )
@@
     )
   )
-  (dimension 46.99 (width 0.3) (layer Dwgs.User)
-    (gr_text "46.990 mm" (at 144.86 94.615 270) (layer Dwgs.User)
+  (dimension 45.212 (width 0.3) (layer Dwgs.User)
+    (gr_text "1.7800 in" (at 142.066 94.488 270) (layer Dwgs.User)
       (effects (font (size 1.5 1.5) (thickness 0.3)))
     )
-    (feature1 (pts (xy 138.43 118.11) (xy 146.21 118.11)))
-    (feature2 (pts (xy 138.43 71.12) (xy 146.21 71.12)))
-    (crossbar (pts (xy 143.51 71.12) (xy 143.51 118.11)))
-    (arrow1a (pts (xy 143.51 118.11) (xy 142.923579 116.983496)))
-    (arrow1b (pts (xy 143.51 118.11) (xy 144.096421 116.983496)))
-    (arrow2a (pts (xy 143.51 71.12) (xy 142.923579 72.246504)))
-    (arrow2b (pts (xy 143.51 71.12) (xy 144.096421 72.246504)))
-  )
-  (dimension 27.94 (width 0.3) (layer Dwgs.User)
-    (gr_text "27.940 mm" (at 124.46 66.468) (layer Dwgs.User)
+    (feature1 (pts (xy 136.906 117.094) (xy 143.416 117.094)))
+    (feature2 (pts (xy 136.906 71.882) (xy 143.416 71.882)))
+    (crossbar (pts (xy 140.716 71.882) (xy 140.716 117.094)))
+    (arrow1a (pts (xy 140.716 117.094) (xy 140.129579 115.967496)))
+    (arrow1b (pts (xy 140.716 117.094) (xy 141.302421 115.967496)))
+    (arrow2a (pts (xy 140.716 71.882) (xy 140.129579 73.008504)))
+    (arrow2b (pts (xy 140.716 71.882) (xy 141.302421 73.008504)))
+  )
+  (dimension 24.384 (width 0.3) (layer Dwgs.User)
+    (gr_text "0.9600 in" (at 124.714 66.468) (layer Dwgs.User)
       (effects (font (size 1.5 1.5) (thickness 0.3)))
     )
-    (feature1 (pts (xy 110.49 71.12) (xy 110.49 65.118)))
-    (feature2 (pts (xy 138.43 71.12) (xy 138.43 65.118)))
-    (crossbar (pts (xy 138.43 67.818) (xy 110.49 67.818)))
-    (arrow1a (pts (xy 110.49 67.818) (xy 111.616504 67.231579)))
-    (arrow1b (pts (xy 110.49 67.818) (xy 111.616504 68.404421)))
-    (arrow2a (pts (xy 138.43 67.818) (xy 137.303496 67.231579)))
-    (arrow2b (pts (xy 138.43 67.818) (xy 137.303496 68.404421)))
-  )
-  (gr_line (start 110.49 118.11) (end 110.49 71.12) (angle 90) (layer Edge.Cuts) (width 0.001))
-  (gr_line (start 138.43 118.11) (end 110.49 118.11) (angle 90) (layer Edge.Cuts) (width 0.001))
-  (gr_line (start 138.43 71.12) (end 138.43 118.11) (angle 90) (layer Edge.Cuts) (width 0.001))
-  (gr_line (start 110.49 71.12) (end 138.43 71.12) (angle 90) (layer Edge.Cuts) (width 0.001))
+    (feature1 (pts (xy 136.906 71.882) (xy 136.906 65.118)))
+    (feature2 (pts (xy 112.522 71.882) (xy 112.522 65.118)))
+    (crossbar (pts (xy 112.522 67.818) (xy 136.906 67.818)))
+    (arrow1a (pts (xy 136.906 67.818) (xy 135.779496 68.404421)))
+    (arrow1b (pts (xy 136.906 67.818) (xy 135.779496 67.231579)))
+    (arrow2a (pts (xy 112.522 67.818) (xy 113.648504 68.404421)))
+    (arrow2b (pts (xy 112.522 67.818) (xy 113.648504 67.231579)))
+  )
+  (gr_line (start 112.522 72.644) (end 112.522 72.39) (angle 90) (layer Edge.Cuts) (width 0.001))
+  (gr_line (start 112.522 71.882) (end 112.522 72.644) (angle 90) (layer Edge.Cuts) (width 0.001))
+  (gr_line (start 136.906 71.882) (end 112.522 71.882) (angle 90) (layer Edge.Cuts) (width 0.001))
+  (gr_line (start 136.906 117.094) (end 136.906 71.882) (angle 90) (layer Edge.Cuts) (width 0.001))
+  (gr_line (start 112.522 117.094) (end 136.906 117.094) (angle 90) (layer Edge.Cuts) (width 0.001))
+  (gr_line (start 112.522 72.136) (end 112.522 117.094) (angle 90) (layer Edge.Cuts) (width 0.001))
   (segment (start 115.316 76.708) (end 115.062 76.708) (width 0.25) (layer F.Cu) (net 1))
   (segment (start 115.062 76.708) (end 114.046 78.994) (width 0.25) (layer F.Cu) (net 1))
@@
   (segment (start 115.824 89.916) (end 115.824 88.9) (width 0.25) (layer B.Cu) (net 12))
   (via (at 115.824 89.916) (size 0.6) (drill 0.4) (layers F.Cu B.Cu) (net 12))
+  (zone (net 1) (net_name GND) (layer F.Cu) (hatch edge 0.508)
+    (connect_pads (clearance 0.508))
+    (min_thickness 0.254)
+    (fill yes (arc_segments 16) (thermal_gap 0.508) (thermal_bridge_width 0.508))
+    (polygon
+      (pts
+        (xy 136.906 117.094) (xy 112.522 117.094) (xy 112.522 71.882) (xy 136.906 71.882) (xy 136.906 117.094)
+      )
+    )
+  )
   (zone (net 1) (net_name GND) (layer B.Cu) (hatch edge 0.508)
     (connect_pads (clearance 0.508))
@@
     (polygon
       (pts
-        (xy 138.43 118.11) (xy 110.49 118.11) (xy 110.49 71.12) (xy 138.43 71.12)
+        (xy 136.906 117.094) (xy 112.522 117.094) (xy 112.522 71.882) (xy 136.906 71.882) (xy 136.906 117.094)
       )
     )
-  )
-  (zone (net 1) (net_name GND) (layer F.Cu) (hatch edge 0.508)
-    (connect_pads (clearance 0.508))
-    (min_thickness 0.254)
-    (fill yes (arc_segments 16) (thermal_gap 0.508) (thermal_bridge_width 0.508))
-    (polygon
-      (pts
-        (xy 138.43 118.11) (xy 110.49 118.11) (xy 110.49 71.12) (xy 138.43 71.12)
-      )
-    )

Commit message: Sending this to the FAB, after opening and checking.
V1
Other:
- net class Default: via_dia 0.6 -> 0.6858; via_drill 0.4 -> 0.3302
- rule via_min_drill: 0.3 -> 0.3302
- rule via_min_size: 0.4 -> 0.6858
